Commit message: Added basic Gazebo sim

File: description/robot_core.urdf.xacro (robot description, xacro)
@@ -6,24 +6,4 @@
     <!-- 베이스 링크: 로봇의 기준 프레임 (Base link: robot reference frame) -->
     <link name="base_link">
-        <!--
-        <visual>
-            <origin xyz="0 0 0" rpy="0 0 0" />
-            <geometry>
-            </geometry>
-            <material name="material_name">
-                <color rgba="1 1 1 1" />
-            </material>
-        </visual>
-        <collision>
-            <origin xyz="0 0 0" rpy="0 0 0" />
-            <geometry>
-            </geometry>
-        </collision>
-        <inertial>
-            <mass value="1.0" />
-            <origin xyz="0 0 0" />
-            <inertia ixx="1.0" ixy="0.0" ixz="0.0" iyy="1.0" iyz="0.0" izz="1.0" />
-        </inertial>
-        -->
     </link>
     <!-- 베이스와 섀시를 연결하는 고정 조인트 (Fixed joint: base to chassis) -->
@@ -52,56 +32,7 @@
         </xacro:inertial_box>
     </link>
-    <!-- 좌측 앞바퀴 조인트 (Left front wheel joint) -->
-    <joint name="left_front_wheel_joint" type="continuous">
-        <parent link="chassis_link" />
-        <child link="left_front_wheel_link" />
-        <origin xyz="0.45 0.15 0" rpy="-${pi/2} 0 0" />
-        <axis xyz="0 0 1" />
-    </joint>
-    <!-- 좌측 앞바퀴 링크 (Left front wheel link) -->
-    <link name="left_front_wheel_link">
-        <visual>
-            <origin xyz="0 0 0" rpy="0 0 0" />
-            <geometry>
-                <cylinder radius="0.075" length="0.0375" />
-            </geometry>
-            <material name="black" />
-        </visual>
-        <collision>
-            <origin xyz="0 0 0" rpy="0 0 0" />
-            <geometry>
-                <cylinder radius="0.075" length="0.0375" />
-            </geometry>
-        </collision>
-            <xacro:inertial_cylinder mass="1.0" radius="0.075" length="0.0375">
-            <origin xyz="0 0 0" rpy="0 0 0" />
-        </xacro:inertial_cylinder>
-    </link>
-    <!-- 우측 앞바퀴 조인트 (Right front wheel joint) -->
-    <joint name="right_front_wheel_joint" type="continuous">
-        <parent link="chassis_link" />
-        <child link="right_front_wheel_link" />
-        <origin xyz="0.45 -0.15 0" rpy="-${pi/2} 0 0" />
-        <axis xyz="0 0 1" />
-    </joint>
-    <!-- 우측 앞바퀴 링크 (Right front wheel link) -->
-    <link name="right_front_wheel_link">
-        <visual>
-            <origin xyz="0 0 0" rpy="0 0 0" />
-            <geometry>
-                <cylinder radius="0.075" length="0.0375" />
-            </geometry>
-            <material name="black" />
-        </visual>
-        <collision>
-            <origin xyz="0 0 0" rpy="0 0 0" />
-            <geometry>
-                <cylinder radius="0.075" length="0.0375" />
-            </geometry>
-        </collision>
-        <xacro:inertial_cylinder mass="1.0" radius="0.075" length="0.0375">
-            <origin xyz="0 0 0" rpy="0 0 0" />
-        </xacro:inertial_cylinder>
-    </link>
+    <gazebo reference="chassis_link">
+        <material>Gazebo/White</material>
+    </gazebo>
     <!-- 좌측 뒷바퀴 조인트 (Left rear wheel joint) -->
     <joint name="left_rear_wheel_joint" type="continuous">
@@ -130,4 +61,7 @@
         </xacro:inertial_cylinder>
     </link>
+    <gazebo reference="left_rear_wheel_link">
+        <material>Gazebo/Black</material>
+    </gazebo>
     <!-- 우측 뒷바퀴 조인트 (Right rear wheel joint) -->
     <joint name="right_rear_wheel_joint" type="continuous">
@@ -156,3 +90,96 @@
         </xacro:inertial_cylinder>
     </link>
+    <gazebo reference="right_rear_wheel_link">
+        <material>Gazebo/Black</material>
+    </gazebo>
+    <!-- 전면 캐스터 휠 추가 (Front caster wheel) -->
+    <joint name="front_caster_joint" type="fixed">
+        <parent link="chassis_link" />
+        <child link="front_caster_link" />
+        <origin xyz="0.45 0 0" rpy="0 0 0" />
+    </joint>
+    <link name="front_caster_link">
+        <visual>
+            <origin xyz="0 0 0" rpy="0 0 0" />
+            <geometry>
+                <sphere radius="0.06" />
+            </geometry>
+            <material name="black" />
+        </visual>
+        <collision>
+            <origin xyz="0 0 0" rpy="0 0 0" />
+            <geometry>
+                <sphere radius="0.06" />
+            </geometry>
+        </collision>
+        <xacro:inertial_sphere mass="0.5" radius="0.06">
+            <origin xyz="0 0 0" rpy="0 0 0" />
+        </xacro:inertial_sphere>
+    </link>
+    <gazebo reference="front_caster_link">
+        <material>Gazebo/Black</material>
+        <mu1 value="0.001" />
+        <mu2 value="0.001" />
+    </gazebo>
+    <!-- 앞바퀴(좌/우) 관련 부분 주석처리: XML 주석 중첩 오류 수정 -->
+    <!--
+    좌측 앞바퀴 조인트 (Left front wheel joint)
+    <joint name="left_front_wheel_joint" type="continuous">
+        <parent link="chassis_link" />
+        <child link="left_front_wheel_link" />
+        <origin xyz="0.45 0.15 0" rpy="-${pi/2} 0 0" />
+        <axis xyz="0 0 1" />
+    </joint>
+    좌측 앞바퀴 링크 (Left front wheel link)
+    <link name="left_front_wheel_link">
+        <visual>
+            <origin xyz="0 0 0" rpy="0 0 0" />
+            <geometry>
+                <cylinder radius="0.075" length="0.0375" />
+            </geometry>
+            <material name="black" />
+        </visual>
+        <collision>
+            <origin xyz="0 0 0" rpy="0 0 0" />
+            <geometry>
+                <cylinder radius="0.075" length="0.0375" />
+            </geometry>
+        </collision>
+        <xacro:inertial_cylinder mass="1.0" radius="0.075" length="0.0375">
+            <origin xyz="0 0 0" rpy="0 0 0" />
+        </xacro:inertial_cylinder>
+    </link>
+    <gazebo reference="left_front_wheel_link">
+        <material>Gazebo/Black</material>
+    </gazebo>
+    우측 앞바퀴 조인트 (Right front wheel joint)
+    <joint name="right_front_wheel_joint" type="continuous">
+        <parent link="chassis_link" />
+        <child link="right_front_wheel_link" />
+        <origin xyz="0.45 -0.15 0" rpy="-${pi/2} 0 0" />
+        <axis xyz="0 0 1" />
+    </joint>
+    우측 앞바퀴 링크 (Right front wheel link)
+    <link name="right_front_wheel_link">
+        <visual>
+            <origin xyz="0 0 0" rpy="0 0 0" />
+            <geometry>
+                <cylinder radius="0.075" length="0.0375" />
+            </geometry>
+            <material name="black" />
+        </visual>
+        <collision>
+            <origin xyz="0 0 0" rpy="0 0 0" />
+            <geometry>
+                <cylinder radius="0.075" length="0.0375" />
+            </geometry>
+        </collision>
+        <xacro:inertial_cylinder mass="1.0" radius="0.075" length="0.0375">
+            <origin xyz="0 0 0" rpy="0 0 0" />
+        </xacro:inertial_cylinder>
+    </link>
+    <gazebo reference="right_front_wheel_link">
+        <material>Gazebo/Black</material>
+    </gazebo>
+    -->
 </robot>
