Commit message: Add simulated lidar

File: description/robot.urdf.xacro (robot description, xacro)
@@ -3,3 +3,4 @@
     <xacro:include filename="robot_core.urdf.xacro" />
     <xacro:include filename="gazebo_control.urdf.xacro" />
+    <xacro:include filename="lidar.urdf.xacro" />
 </robot>

File: description/robot_core.urdf.xacro (robot description, xacro)
@@ -103,5 +103,5 @@
             <origin xyz="0 0 0" rpy="0 0 0" />
             <geometry>
-                <sphere radius="0.06" />
+                <sphere radius="0.075" />
             </geometry>
             <material name="black" />
@@ -110,8 +110,8 @@
             <origin xyz="0 0 0" rpy="0 0 0" />
             <geometry>
-                <sphere radius="0.06" />
+                <sphere radius="0.075" />
             </geometry>
         </collision>
-        <xacro:inertial_sphere mass="0.5" radius="0.06">
+        <xacro:inertial_sphere mass="0.5" radius="0.075">
             <origin xyz="0 0 0" rpy="0 0 0" />
         </xacro:inertial_sphere>
