Commit message: Add initial ros2_control code

File: description/color.urdf.xacro (robot description, xacro)
@@ -1,5 +1,4 @@
 <?xml version="1.0"?>
 <robot xmlns:xacro="http://www.ros.org/wiki/xacro">
-    <!-- 무지개색 계열 -->
     <material name="red">
         <color rgba="1 0 0 1" />
@@ -23,5 +22,4 @@
         <color rgba="0.5 0 0.5 1" />
     </material>
-    <!-- 흑백/회색 계열 -->
     <material name="white">
         <color rgba="1 1 1 1" />
@@ -39,5 +37,4 @@
         <color rgba="0 0 0 1" />
     </material>
-    <!-- 금속/특수색 -->
     <material name="gold">
         <color rgba="1 0.84 0 1" />
@@ -49,5 +46,4 @@
         <color rgba="0.8 0.5 0.2 1" />
     </material>
-    <!-- 기타/파스텔/알파벳순 -->
     <material name="aqua">
         <color rgba="0 1 1 1" />

File: description/depth_camera.urdf.xacro (robot description, xacro)
@@ -49,11 +49,11 @@
                 <clip>
                     <near>0.05</near>
-                    <far>8.0</far>
+                    <far>12.0</far>
                 </clip>
             </camera>
             <plugin name="camera_controller" filename="libgazebo_ros_camera.so">
                 <frame_name>camera_link_optical</frame_name>
-                <min_depth>0.1</min_depth>
-                <max_depth>100.0</max_depth>
+                <min_depth>0.05</min_depth>
+                <max_depth>12.0</max_depth>
             </plugin>
         </sensor>

File: description/gazebo_control.urdf.xacro (robot description, xacro)
@@ -1,24 +1,14 @@
 <?xml version="1.0"?>
 <robot xmlns:xacro="http://www.ros.org/wiki/xacro">
-  <!-- Gazebo 시뮬레이터용 diff_drive 플러그인 설정 -->
   <gazebo>
     <plugin name="diff_drive_controller" filename="libgazebo_ros_diff_drive.so">
-      <!-- 좌측 바퀴 조인트(앞/뒤) -->
       <left_joint>left_rear_wheel_joint</left_joint>
-      <!-- 우측 바퀴 조인트(앞/뒤) -->
       <right_joint>right_rear_wheel_joint</right_joint>
-      <!-- 바퀴 간 거리 (m) -->
       <wheel_separation>0.3</wheel_separation>
-      <!-- 바퀴 지름 (m) -->
-      <wheel_diameter>0.15</wheel_diameter>
-      <!-- 최대 바퀴 토크 -->
+      <wheel_diameter>0.075</wheel_diameter>
       <max_wheel_torque>200</max_wheel_torque>
-      <!-- 최대 바퀴 가속도 -->
       <max_wheel_acceleration>10.0</max_wheel_acceleration>
-      <!-- 오도메트리 프레임 -->
       <odometry_frame>odom</odometry_frame>
-      <!-- 로봇 베이스 프레임 -->
       <robot_base_frame>base_link</robot_base_frame>
-      <!-- 오도메트리 및 TF publish 설정 -->
       <publish_odom>true</publish_odom>
       <publish_odom_tf>true</publish_odom_tf>

File: description/robot.urdf.xacro (robot description, xacro)
@@ -2,5 +2,6 @@
 <robot xmlns:xacro="http://www.ros.org/wiki/xacro"  name="robot">
     <xacro:include filename="robot_core.urdf.xacro" />
-    <xacro:include filename="gazebo_control.urdf.xacro" />
+    <!-- <xacro:include filename="gazebo_control.urdf.xacro" /> -->
+    <xacro:include filename="ros2_control.urdf.xacro" />
     <xacro:include filename="lidar.urdf.xacro" />
     <!-- <xacro:include filename="camera.urdf.xacro" /> -->

File: description/robot_core.urdf.xacro (robot description, xacro)
@@ -1,11 +1,8 @@
 <?xml version="1.0"?>
 <robot xmlns:xacro="http://www.ros.org/wiki/xacro">
-    <!-- 색상 정의 파일 포함 (Include color definitions) -->
     <xacro:include filename="color.urdf.xacro" />
     <xacro:include filename="inertia.urdf.xacro" />
-    <!-- 베이스 링크: 로봇의 기준 프레임 (Base link: robot reference frame) -->
     <link name="base_link">
     </link>
-    <!-- 베이스와 섀시를 연결하는 고정 조인트 (Fixed joint: base to chassis) -->
     <joint name="chassis_joint" type="fixed">
         <parent link="base_link" />
@@ -13,5 +10,4 @@
         <origin xyz="-0.3 0 0" rpy="0 0 0" />
     </joint>
-    <!-- 섀시 링크 (Chassis link: robot body) -->
     <link name="chassis_link">
         <visual>
@@ -35,5 +31,4 @@
         <material>Gazebo/White</material>
     </gazebo>
-    <!-- 좌측 뒷바퀴 조인트 (Left rear wheel joint) -->
     <joint name="left_rear_wheel_joint" type="continuous">
         <parent link="chassis_link" />
@@ -42,5 +37,4 @@
         <axis xyz="0 0 1" />
     </joint>
-    <!-- 좌측 뒷바퀴 링크 (Left rear wheel link) -->
     <link name="left_rear_wheel_link">
         <visual>
@@ -64,5 +58,4 @@
         <material>Gazebo/Black</material>
     </gazebo>
-    <!-- 우측 뒷바퀴 조인트 (Right rear wheel joint) -->
     <joint name="right_rear_wheel_joint" type="continuous">
         <parent link="chassis_link" />
@@ -71,5 +64,4 @@
         <axis xyz="0 0 1" />
     </joint>
-    <!-- 우측 뒷바퀴 링크 (Right rear wheel link) -->
     <link name="right_rear_wheel_link">
         <visual>
@@ -93,5 +85,4 @@
         <material>Gazebo/Black</material>
     </gazebo>
-    <!-- 전면 캐스터 휠 추가 (Front caster wheel) -->
     <joint name="front_caster_joint" type="fixed">
         <parent link="chassis_link" />
@@ -122,64 +113,3 @@
         <mu2 value="0.001" />
     </gazebo>
-    <!-- 앞바퀴(좌/우) 관련 부분 주석처리: XML 주석 중첩 오류 수정 -->
-    <!--
-    좌측 앞바퀴 조인트 (Left front wheel joint)
-    <joint name="left_front_wheel_joint" type="continuous">
-        <parent link="chassis_link" />
-        <child link="left_front_wheel_link" />
-        <origin xyz="0.45 0.15 0" rpy="-${pi/2} 0 0" />
-        <axis xyz="0 0 1" />
-    </joint>
-    좌측 앞바퀴 링크 (Left front wheel link)
-    <link name="left_front_wheel_link">
-        <visual>
-            <origin xyz="0 0 0" rpy="0 0 0" />
-            <geometry>
-                <cylinder radius="0.075" length="0.0375" />
-            </geometry>
-            <material name="black" />
-        </visual>
-        <collision>
-            <origin xyz="0 0 0" rpy="0 0 0" />
-            <geometry>
-                <cylinder radius="0.075" length="0.0375" />
-            </geometry>
-        </collision>
-        <xacro:inertial_cylinder mass="1.0" radius="0.075" length="0.0375">
-            <origin xyz="0 0 0" rpy="0 0 0" />
-        </xacro:inertial_cylinder>
-    </link>
-    <gazebo reference="left_front_wheel_link">
-        <material>Gazebo/Black</material>
-    </gazebo>
-    우측 앞바퀴 조인트 (Right front wheel joint)
-    <joint name="right_front_wheel_joint" type="continuous">
-        <parent link="chassis_link" />
-        <child link="right_front_wheel_link" />
-        <origin xyz="0.45 -0.15 0" rpy="-${pi/2} 0 0" />
-        <axis xyz="0 0 1" />
-    </joint>
-    우측 앞바퀴 링크 (Right front wheel link)
-    <link name="right_front_wheel_link">
-        <visual>
-            <origin xyz="0 0 0" rpy="0 0 0" />
-            <geometry>
-                <cylinder radius="0.075" length="0.0375" />
-            </geometry>
-            <material name="black" />
-        </visual>
-        <collision>
-            <origin xyz="0 0 0" rpy="0 0 0" />
-            <geometry>
-                <cylinder radius="0.075" length="0.0375" />
-            </geometry>
-        </collision>
-        <xacro:inertial_cylinder mass="1.0" radius="0.075" length="0.0375">
-            <origin xyz="0 0 0" rpy="0 0 0" />
-        </xacro:inertial_cylinder>
-    </link>
-    <gazebo reference="right_front_wheel_link">
-        <material>Gazebo/Black</material>
-    </gazebo>
-    -->
 </robot>
