Commit message: Add SLAM stuff

File: description/camera.urdf.xacro (robot description, xacro)
@@ -39,5 +39,5 @@
             <pose> 0 0 0 0 0 0 </pose>
             <visualize>true</visualize>
-            <update_rate>100</update_rate>
+            <update_rate>20</update_rate>
             <camera>
                 <horizontal_fov>1.089</horizontal_fov>

File: description/depth_camera.urdf.xacro (robot description, xacro)
@@ -39,5 +39,5 @@
             <pose> 0 0 0 0 0 0 </pose>
             <visualize>true</visualize>
-            <update_rate>100</update_rate>
+            <update_rate>20</update_rate>
             <camera>
                 <horizontal_fov>1.089</horizontal_fov>

File: description/lidar.urdf.xacro (robot description, xacro)
@@ -30,5 +30,5 @@
             <pose> 0 0 0 0 0 0 </pose>
             <visualize>false</visualize>
-            <update_rate>100</update_rate>
+            <update_rate>20</update_rate>
             <ray>
                 <scan>
@@ -41,5 +41,5 @@
                 </scan>
                 <range>
-                    <min>0.3</min>
+                    <min>0.06</min>
                     <max>12</max>
                     <resolution>0.01</resolution>

File: description/robot_core.urdf.xacro (robot description, xacro)
@@ -4,4 +4,11 @@
     <xacro:include filename="inertia.urdf.xacro" />
     <link name="base_link">
+    </link>
+    <joint name="base_footprint_joint" type="fixed">
+        <parent link="base_link"/>
+        <child link="base_footprint"/>
+        <origin xyz="0 0 0" rpy="0 0 0"/>
+    </joint>
+    <link name="base_footprint">
     </link>
     <joint name="chassis_joint" type="fixed">
